Commit message: remove one thirdparty mesh dependency

File: cabot_description/urdf/sensors/_d435.urdf.xacro (robot description, xacro)
@@ -50,6 +50,5 @@
         <geometry>
           <!-- <box size="${d435_cam_width} ${d435_cam_height} ${d435_cam_depth}"/> -->
-          <mesh filename="package://cabot_description/meshes/sensors/d435.dae" />
-          <!--<mesh filename="package://realsense2_description/meshes/d435/d435.dae" />-->
+          <mesh filename="package://realsense2_description/meshes/d435.dae" />
         </geometry>
         <material name="${name}_aluminum"/>
