Commit message: update cabot_description pkg to v2.0 update LICENSE file

File: cabot_description/robots/cabot1-f.urdf.xacro (robot description, xacro)
@@ -19,14 +19,20 @@
 -->
 <robot name="cabot" xmlns:xacro="http://ros.org/wiki/xacro">
+  <!-- robot rotation center offset -->
+  <xacro:arg name="offset" default="0" />
+  <!-- flag to extend hokuyo lidar range in simulation -->
   <xacro:arg name="extended" default="0" />
-  <xacro:arg name="publish_tf" default="1" />
-  <xacro:arg name="offset" default="0" />
-  <xacro:include filename="$(find cabot_description)/urdf/cabot-e_description.urdf" />
+  <!-- include xacro macros -->
+  <xacro:include filename="$(find cabot_description)/urdf/cabot1-f_description.urdf" />
   <xacro:include filename="$(find cabot_description)/urdf/sensors/hokuyo_ust_20lx.urdf.xacro"/>
   <xacro:include filename="$(find cabot_description)/urdf/sensors/zed.urdf.xacro"/>
+  <!-- content -->
+  <!-- cabot description -->
+  <cabot offset="$(arg offset)"/>
+  <!-- add link to lidar and camera -->
   <link name="lidar_link">
   </link>
   <joint name="lidar_base" type="fixed">
-    <origin xyz="0.125 0.0 0.425" rpy="0 0 0"/>
+    <origin xyz="0.25 0.0 0.10" rpy="0 0 0"/>
     <parent link="base_link"/>
     <child link="lidar_link"/>
@@ -35,15 +41,10 @@
   </link>
   <joint name="camera_base" type="fixed">
-    <origin xyz="0.025 0.0 0.77" rpy="0 0 0"/>
+    <origin xyz="0.025 0.0 0.755" rpy="0 0 0"/>
     <parent link="base_link"/>
     <child link="camera_link"/>
   </joint>
-  <cabot publish_tf="$(arg publish_tf)" offset="$(arg offset)"/>
-  <xacro:unless value="$(arg extended)">
-    <sensor_hokuyo_ust_20lx parent="lidar_link"/>
-  </xacro:unless>
-  <xacro:if value="$(arg extended)">
-    <sensor_hokuyo_ust_20lx parent="lidar_link" sample="1440" min_angle="-3.5" max_angle="2.2" />
-  </xacro:if>
+  <!-- lidar and zed camera description -->
+  <sensor_hokuyo_ust_20lx parent="lidar_link" extended="$(arg extended)"/>
   <sensor_zed parent="camera_link"/>
 </robot>

File: cabot_description/robots/cabot2-s1.urdf.xacro (robot description, xacro)
@@ -19,30 +19,41 @@
 -->
 <robot name="cabot" xmlns:xacro="http://ros.org/wiki/xacro">
+  <!-- robot rotation center offset -->
+  <xacro:arg name="offset" default="0" />
+  <!-- flag to extend hokuyo lidar range in simulation -->
   <xacro:arg name="extended" default="0" />
-  <xacro:arg name="offset" default="0" />
-  <xacro:include filename="$(find cabot_description)/urdf/cabot-f_description.urdf" />
+  <xacro:include filename="$(find cabot_description)/urdf/cabot2-s1_description.urdf" />
   <xacro:include filename="$(find cabot_description)/urdf/sensors/hokuyo_ust_20lx.urdf.xacro"/>
   <xacro:include filename="$(find cabot_description)/urdf/sensors/zed.urdf.xacro"/>
+  <!-- cabot description -->
+  <cabot offset="$(arg offset)"/>
+  <!-- add link to lidar and camera -->
   <link name="lidar_link">
   </link>
   <joint name="lidar_base" type="fixed">
-    <origin xyz="0.25 0.0 0.10" rpy="0 0 0"/>
-    <parent link="base_link"/>
-    <child link="lidar_link"/>
-  </joint>
+      <origin xyz="0.15 0.0 0.12" rpy="0 0 0"/>
+      <parent link="base_link"/>
+      <child link="lidar_link"/>
+    </joint>
   <link name="camera_link">
   </link>
   <joint name="camera_base" type="fixed">
-    <origin xyz="0.025 0.0 0.77" rpy="0 0 0"/>
-    <parent link="base_link"/>
-    <child link="camera_link"/>
+      <origin xyz="0.0 0.0 0.755" rpy="0 0 0"/>
+      <parent link="base_link"/>
+      <child link="camera_link"/>
   </joint>
-  <cabot offset="$(arg offset)"/>
-  <xacro:unless value="$(arg extended)">
-    <sensor_hokuyo_ust_20lx parent="lidar_link"/>
-  </xacro:unless>
-  <xacro:if value="$(arg extended)">
-    <sensor_hokuyo_ust_20lx parent="lidar_link" sample="1440" min_angle="-3.5" max_angle="2.2" />
-  </xacro:if>
+  <!--
+  <sensor_hokuyo_ust_20lx parent="lidar_link" offset="0"/>
+  -->
   <sensor_zed parent="camera_link"/>
+  <!-- VLP-16 -->
+  <xacro:arg name="gpu" default="true"/>
+  <xacro:property name="gpu" value="$(arg gpu)" />
+  <xacro:include filename="$(find velodyne_description)/urdf/VLP-16.urdf.xacro"/>
+  <VLP-16 parent="base_link" name="velodyne" topic="/velodyne_points" hz="10" gpu="${gpu}">
+    <origin xyz="0 0 0.5" rpy="0 0 0" />
+  </VLP-16>
+  <!-- IMU sensor -->
+  <xacro:include filename="$(find cabot_description)/urdf/sensors/imu_sensor.urdf.xacro"/>
+  <imu_macro prefix="imu" frame="imu_frame"/>
 </robot>

File: cabot_description/urdf/sensors/hokuyo_ust_20lx.urdf.xacro (robot description, xacro)
@@ -19,69 +19,77 @@
 -->
 <robot name="sensor_hokuyo_ust_20lx"
-  xmlns:xacro="http://ros.org/wiki/xacro">
-  <xacro:macro name="sensor_hokuyo_ust_20lx_gazebo" params="sample:=1080 min_angle:=-1.57 max_angle:=1.57">
-    <gazebo reference="hokuyo_link">
-      <sensor type="ray" name="head_hokuyo_sensor">
-        <pose>0 0 0 0 0 0</pose>
-        <visualize>true</visualize>
-        <update_rate>40</update_rate>
-        <ray>
-          <scan>
-            <horizontal>
-              <samples>${sample}</samples> <!-- sample per 0.25 degree -->
-              <resolution>0.25</resolution>
-              <min_angle>${min_angle}</min_angle>
-              <max_angle>${max_angle}</max_angle>
-            </horizontal>
-          </scan>
-          <range>
-            <min>0.06</min>
-            <max>20.0</max>
-            <resolution>0.01</resolution>
-          </range>
-          <noise>
-            <type>gaussian</type>
-            <!-- Noise parameters based on published spec for Hokuyo laser
+	xmlns:xacro="http://ros.org/wiki/xacro">
+	<xacro:macro name="turtlebot_sim_laser_range_finder" params="samples:=1080 resolution:=0.25 min_angle:=-1.57 max_angle:=1.57">
+		<gazebo reference="hokuyo_link">
+			<sensor type="ray" name="head_hokuyo_sensor">
+				<pose>0 0 0 0 0 0</pose>
+				<visualize>true</visualize>
+				<update_rate>10</update_rate>
+				<ray>
+					<scan>
+						<horizontal>
+							<samples>${samples}</samples>
+							<resolution>${resolution}</resolution>
+							<min_angle>${min_angle}</min_angle>
+							<max_angle>${max_angle}</max_angle>
+						</horizontal>
+					</scan>
+					<range>
+						<min>0.06</min>
+						<max>20.0</max>
+						<resolution>0.01</resolution>
+					</range>
+					<noise>
+						<type>gaussian</type>
+						<!-- Noise parameters based on published spec for Hokuyo laser
 		 achieving "+-30mm" accuracy at range < 10m.  A mean of 0.0m and
 		 stddev of 0.01m will put 99.7% of samples within 0.03m of the true
 		 reading. -->
-            <!-- x 1.3 for "+-40mm" accuracy for 20lx. Original value is 0.01 -->
-            <mean>0.0</mean>
-            <stddev>0.013</stddev>
-          </noise>
-        </ray>
-        <plugin name="gazebo_ros_head_hokuyo_controller" filename="libgazebo_ros_laser.so">
-          <topicName>scan</topicName>
-          <frameName>hokuyo_link</frameName>
-        </plugin>
-      </sensor>
-    </gazebo>
-  </xacro:macro>
-  <xacro:macro name="sensor_hokuyo_ust_20lx" params="parent offset:=0 sample:=1080 min_angle:=-1.57 max_angle:=1.57">
-    <link name="hokuyo_link">
-      <collision>
-        <origin xyz="0 0 0" rpy="0 0 0"/>
-        <geometry>
-          <box size="0.05 0.05 0.05"/>
-        </geometry>
-      </collision>
-      <visual>
-        <origin xyz="0 0 0" rpy="0 0 0"/>
-        <geometry>
-          <mesh filename="package://cabot_description/meshes/thirdparty/hokuyo.dae"/>
-        </geometry>
-      </visual>
-      <inertial>
-        <mass value="1e-5" />
-        <origin xyz="0 0 0" rpy="0 0 0"/>
-        <inertia ixx="1e-6" ixy="0" ixz="0" iyy="1e-6" iyz="0" izz="1e-6" />
-      </inertial>
-    </link>
-    <joint name="hokuyo_joint" type="fixed">
-      <origin xyz="0.0 ${offset} 0.0" rpy="0 0 0"/>
-      <parent link="${parent}"/>
-      <child link="hokuyo_link"/>
-    </joint>
-    <sensor_hokuyo_ust_20lx_gazebo sample="${sample}" min_angle="${min_angle}" max_angle="${max_angle}" />
-  </xacro:macro>
+						<!-- x 1.3 for "+-40mm" accuracy for 20lx. Original value is 0.01 -->
+						<mean>0.0</mean>
+						<stddev>0.013</stddev>
+					</noise>
+				</ray>
+				<plugin name="gazebo_ros_head_hokuyo_controller" filename="libgazebo_ros_laser.so">
+					<topicName>/scan</topicName>
+					<frameName>hokuyo_link</frameName>
+				</plugin>
+			</sensor>
+		</gazebo>
+	</xacro:macro>
+	<!--xacro:include filename="$(find turtlebot_description)/urdf/turtlebot_properties.urdf.xacro"/-->
+	<xacro:macro name="sensor_hokuyo_ust_20lx" params="parent extended:=0 min_angle:=-1.57 max_angle:=1.57">
+		<link name="hokuyo_link">
+			<collision>
+				<origin xyz="0 0 0" rpy="0 0 0"/>
+				<geometry>
+					<box size="0.05 0.05 0.05"/>
+				</geometry>
+			</collision>
+			<visual>
+				<origin xyz="0 0 0" rpy="0 0 0"/>
+				<geometry>
+					<mesh filename="package://cabot_description/meshes/sensors/hokuyo.dae"/>
+				</geometry>
+			</visual>
+			<inertial>
+				<mass value="1e-5" />
+				<origin xyz="0 0 0" rpy="0 0 0"/>
+				<inertia ixx="1e-6" ixy="0" ixz="0" iyy="1e-6" iyz="0" izz="1e-6" />
+			</inertial>
+		</link>
+		<joint name="hokuyo_joint" type="fixed">
+			<!--<axis xyz="0 0 1" />-->
+			<origin xyz="0.0 0.0 0.0" rpy="0 0 0"/>
+			<parent link="${parent}"/>
+			<child link="hokuyo_link"/>
+		</joint>
+		<!-- Hokuyo sensor for simulation -->
+		<xacro:unless value="$(arg extended)">
+			<turtlebot_sim_laser_range_finder min_angle="${min_angle}" max_angle="${max_angle}"/>
+		</xacro:unless>
+		<xacro:if value="$(arg extended)">
+			<turtlebot_sim_laser_range_finder samples="1440" min_angle="-3.5" max_angle="2.2"/>
+		</xacro:if>
+	</xacro:macro>
 </robot>

Commit message: Add following new features from IBM Research - Tokyo, Accessibility Research Group
- A library for localizing a robot in multi floor environments to support navigating wide areas.
- A library for recognizing surrounding people from images to support navigating in socially acceptable ways.

DCO 1.1 Signed-off-by: Tatsuya Ishihara <tisihara@jp.ibm.com>

File: cabot_description/robots/cabot1-f.urdf.xacro (robot description, xacro)
@@ -1,5 +1,5 @@
 <?xml version="1.0"?>
 <!--
- Copyright (c) 2020  Carnegie Mellon University
+ Copyright (c) 2020 Carnegie Mellon University
  Permission is hereby granted, free of charge, to any person obtaining a copy
  of this software and associated documentation files (the "Software"), to deal

File: cabot_description/robots/cabot2-e2.urdf.xacro (robot description, xacro)
@@ -1,5 +1,5 @@
 <?xml version="1.0"?>
 <!--
- Copyright (c) 2020  Carnegie Mellon University
+ Copyright (c) 2020 Carnegie Mellon University
  Permission is hereby granted, free of charge, to any person obtaining a copy
  of this software and associated documentation files (the "Software"), to deal

File: cabot_description/robots/cabot2-gt1.urdf.xacro (robot description, xacro)
@@ -1,5 +1,5 @@
 <?xml version="1.0"?>
 <!--
- Copyright (c) 2020  Carnegie Mellon University
+ Copyright (c) 2020 Carnegie Mellon University
  Permission is hereby granted, free of charge, to any person obtaining a copy
  of this software and associated documentation files (the "Software"), to deal

File: cabot_description/robots/cabot2-s1.urdf.xacro (robot description, xacro)
@@ -1,5 +1,5 @@
 <?xml version="1.0"?>
 <!--
- Copyright (c) 2020  Carnegie Mellon University
+ Copyright (c) 2020 Carnegie Mellon University
  Permission is hereby granted, free of charge, to any person obtaining a copy
  of this software and associated documentation files (the "Software"), to deal

File: cabot_description/urdf/sensors/_d435.urdf.xacro (robot description, xacro)
@@ -50,5 +50,6 @@
         <geometry>
           <!-- <box size="${d435_cam_width} ${d435_cam_height} ${d435_cam_depth}"/> -->
-          <mesh filename="package://realsense2_description/meshes/d435.dae" />
+          <mesh filename="package://cabot_description/meshes/sensors/d435.dae" />
+          <!--<mesh filename="package://realsense2_description/meshes/d435/d435.dae" />-->
         </geometry>
         <material name="${name}_aluminum"/>

File: cabot_description/urdf/sensors/hokuyo_ust_20lx.urdf.xacro (robot description, xacro)
@@ -1,5 +1,5 @@
 <?xml version="1.0"?>
 <!--
- Copyright (c) 2020  Carnegie Mellon University
+ Copyright (c) 2020 Carnegie Mellon University
  Permission is hereby granted, free of charge, to any person obtaining a copy
  of this software and associated documentation files (the "Software"), to deal

File: cabot_description/urdf/sensors/zed.urdf.xacro (robot description, xacro)
@@ -1,5 +1,5 @@
 <?xml version="1.0"?>
 <!--
- Copyright (c) 2020  Carnegie Mellon University
+ Copyright (c) 2020 Carnegie Mellon University
  Permission is hereby granted, free of charge, to any person obtaining a copy
  of this software and associated documentation files (the "Software"), to deal
