Commit message: roughly update cabot2-ace description and urdf
Signed-off-by: Masayuki Murata <muratams@jp.ibm.com>

File: cabot_description/robots/cabot2-ace.urdf.xacro (robot description, xacro)
@@ -43,5 +43,5 @@
   <joint name="lidar_base" type="fixed">
     <!--<origin xyz="0.15 0.0 0.12" rpy="0 0 0"/>-->
-      <origin xyz="0.02 0.0 0.58" rpy="0 0 1.57"/> <!-- lidar base points to the left direction.-->
+      <origin xyz="0.10 0.0 0.58" rpy="0 0 0"/>
       <parent link="base_link"/>
       <child link="lidar_link"/>

Commit message: update cabot2-ace the body dimensions, lidar position, and imu position
Signed-off-by: Masayuki Murata <muratams@jp.ibm.com>

File: cabot_description/robots/cabot2-ace.urdf.xacro (robot description, xacro)
@@ -42,6 +42,5 @@
   </link>
   <joint name="lidar_base" type="fixed">
-    <!--<origin xyz="0.15 0.0 0.12" rpy="0 0 0"/>-->
-      <origin xyz="0.10 0.0 0.58" rpy="0 0 0"/>
+      <origin xyz="0.10 0.0 0.477" rpy="0 0 0"/> <!-- lidar mount position -->
       <parent link="base_link"/>
       <child link="lidar_link"/>
@@ -82,5 +81,5 @@
     <xacro:VLP-16 parent="lidar_link" name="velodyne" topic="/velodyne_points"
 	    hz="10" gpu="${gpu}" min_range="0.3">
-      <origin xyz="0 0 0.0" rpy="0 0 0" />
+      <origin xyz="0 0 0" rpy="0 0 0" />
     </xacro:VLP-16>
   </xacro:if>

Commit message: adjust cabot2-ace urdf model
Signed-off-by: Daisuke Sato <dsato@jp.ibm.com>

File: cabot_description/robots/cabot2-ace.urdf.xacro (robot description, xacro)
@@ -35,4 +35,5 @@
   <xacro:include filename="$(find cabot_description)/urdf/sensors/imu_sensor.urdf.xacro"/>
   <xacro:include filename="$(find cabot_description)/urdf/sensors/_d435.urdf.xacro"/>
+  <xacro:include filename="$(find cabot_description)/urdf/sensors/_d455.urdf.xacro"/>
   <!-- content -->
   <!-- cabot description -->
@@ -45,10 +46,17 @@
       <parent link="base_link"/>
       <child link="lidar_link"/>
-    </joint>
+  </joint>
+  <link name="camera_link">
+  </link>
+  <joint name="camera_base" type="fixed">
+      <origin xyz="0.19 0.0 0.45" rpy="0 0 0"/>
+      <parent link="base_link"/>
+      <child link="camera_link"/>
+  </joint>
   <link name="rs1_link">
   </link>
   <joint name="rs1_base" type="fixed">
       <origin xyz="0 0 0" rpy="0 0 0"/>
-      <parent link="base_link"/>
+      <parent link="camera_link"/>
       <child link="rs1_link"/>
   </joint>
@@ -56,6 +64,6 @@
   </link>
   <joint name="rs2_base" type="fixed">
-      <origin xyz="-0.01 -0.09 0.01" rpy="-0.3 0.0 0.0"/>
-      <parent link="base_link"/>
+      <origin xyz="-0.04 -0.10 0.0" rpy="0 0.0 ${-75.0/180.0*3.14}"/>
+      <parent link="camera_link"/>
       <child link="rs2_link"/>
   </joint>
@@ -63,6 +71,6 @@
   </link>
   <joint name="rs3_base" type="fixed">
-      <origin xyz="-0.01 0.08 0.01" rpy="0.3 0.0 3.14"/>
-      <parent link="base_link"/>
+      <origin xyz="-0.04 0.10 0.025" rpy="3.14 0.0 ${75.0/180.0*3.14}"/>
+      <parent link="camera_link"/>
       <child link="rs3_link"/>
   </joint>
@@ -86,15 +94,15 @@
   <!-- RealSense D435 -->
   <xacro:if value="${camera_type=='realsense'}">
-    <xacro:sensor_d435 parent="rs1_link" name="d435_rs1">
+    <xacro:sensor_d455 parent="rs1_link" name="d455_rs1" topics_ns="rs1">
+      <origin xyz="0 0 0" rpy="0 0 0" />
+    </xacro:sensor_d455>
+  </xacro:if>
+  <xacro:if value="${camera_type=='realsense'}">
+    <xacro:sensor_d435 parent="rs2_link" name="d435_rs2" topics_ns="rs2">
       <origin xyz="0 0 0" rpy="0 0 0" />
     </xacro:sensor_d435>
   </xacro:if>
   <xacro:if value="${camera_type=='realsense'}">
-    <xacro:sensor_d435 parent="rs2_link" name="d435_rs2">
-      <origin xyz="0 0 0" rpy="0 0 0" />
-    </xacro:sensor_d435>
-  </xacro:if>
-  <xacro:if value="${camera_type=='realsense'}">
-    <xacro:sensor_d435 parent="rs3_link" name="d435_rs3">
+    <xacro:sensor_d435 parent="rs3_link" name="d435_rs3" topics_ns="rs3">
       <origin xyz="0 0 0" rpy="0 0 0" />
     </xacro:sensor_d435>

Commit message: adjust parameters based on CAD model, add body STL model

File: cabot_description/robots/cabot2-ace.urdf.xacro (robot description, xacro)
@@ -43,5 +43,5 @@
   </link>
   <joint name="lidar_base" type="fixed">
-      <origin xyz="0.10 0.0 0.477" rpy="0 0 0"/> <!-- lidar mount position -->
+      <origin xyz="0.0955 -0.0025 ${0.522-0.038}" rpy="0 0 0"/> <!-- lidar mount position -->
       <parent link="base_link"/>
       <child link="lidar_link"/>
@@ -50,5 +50,5 @@
   </link>
   <joint name="camera_base" type="fixed">
-      <origin xyz="0.19 0.0 0.45" rpy="0 0 0"/>
+      <origin xyz="0.1657 -0.0025 ${0.490285-0.038}" rpy="0 0 0"/>
       <parent link="base_link"/>
       <child link="camera_link"/>
@@ -57,6 +57,6 @@
   </link>
   <joint name="rs1_base" type="fixed">
-      <origin xyz="0 0 0" rpy="0 0 0"/>
-      <parent link="camera_link"/>
+      <origin xyz="0.1657 -0.0025 ${0.490285-0.038}" rpy="0 0 0"/>
+      <parent link="base_link"/>
       <child link="rs1_link"/>
   </joint>
@@ -64,6 +64,6 @@
   </link>
   <joint name="rs2_base" type="fixed">
-      <origin xyz="-0.04 -0.10 0.0" rpy="0 0.0 ${-75.0/180.0*3.14}"/>
-      <parent link="camera_link"/>
+      <origin xyz="0.12843 -0.08815 ${0.49285-0.038}" rpy="0 0 ${-70.0/180.0*3.1415926535}"/>
+      <parent link="base_link"/>
       <child link="rs2_link"/>
   </joint>
@@ -71,6 +71,6 @@
   </link>
   <joint name="rs3_base" type="fixed">
-      <origin xyz="-0.04 0.10 0.025" rpy="3.14 0.0 ${75.0/180.0*3.14}"/>
-      <parent link="camera_link"/>
+      <origin xyz="0.12843 0.083154 ${0.517285-0.038}" rpy="3.1415926535 0 ${70.0/180.0*3.1415926535}"/>
+      <parent link="base_link"/>
       <child link="rs3_link"/>
   </joint>

File: cabot_description/urdf/sensors/_d435.urdf.xacro (robot description, xacro)
@@ -47,5 +47,6 @@
     <link name="${name}_link">
       <visual>
-      <origin xyz="${-d435_cam_depth_px} ${-d435_cam_depth_py} 0" rpy="${M_PI/2} 0 ${M_PI/2}"/>
+      <!--origin xyz="${-d435_cam_depth_px} ${-d435_cam_depth_py} 0" rpy="${M_PI/2} 0 ${M_PI/2}"/-->
+      <origin xyz="0 ${-d435_cam_depth_py} 0" rpy="${M_PI/2} 0 ${M_PI/2}"/>
         <geometry>
           <!-- <box size="${d435_cam_width} ${d435_cam_height} ${d435_cam_depth}"/> -->

File: cabot_description/urdf/sensors/_d455.urdf.xacro (robot description, xacro)
@@ -50,5 +50,5 @@
     <link name="${name}_link">
       <visual>
-      <origin xyz="${-d455_cam_depth_px} ${-d455_cam_depth_py} 0" rpy="${M_PI/2} 0 ${M_PI/2}"/>
+      <origin xyz="0 ${-d455_cam_depth_py} 0" rpy="${M_PI/2} 0 ${M_PI/2}"/>
         <geometry>
           <!-- <box size="${d455_cam_width} ${d455_cam_height} ${d455_cam_depth}"/> -->

Commit message: add a function to use gnss fix to improve localization in outdoor
- add gnss fix callback funtion to multi_floor_manager
- update cartographer version in thirdparty repos
- add a docker service to run rtk
- add an option to launch ublox zed-f9p gnss receiver

Signed-off-by: Masayuki Murata <muratams@jp.ibm.com>

File: cabot_description/robots/cabot2-ace.urdf.xacro (robot description, xacro)
@@ -56,4 +56,12 @@
   <link name="rs1_link">
   </link>
+  <!-- add link to gps--> <!-- lidar + 0.1m in z-direction -->
+  <link name="gps">
+  </link>
+  <joint name="gps_base" type="fixed">
+      <origin xyz="0.0955 0.0 0.68" rpy="0 0 0"/>
+      <parent link="base_link"/>
+      <child link="gps"/>
+  </joint>
   <joint name="rs1_base" type="fixed">
       <origin xyz="0.1657 -0.0025 ${0.490285-0.038}" rpy="0 0 0"/>

File: cabot_description/robots/cabot2-gt1.urdf.xacro (robot description, xacro)
@@ -54,4 +54,12 @@
       <child link="camera_link"/>
   </joint>
+  <!-- add link to gps--> <!-- lidar + 0.1m in z-direction -->
+  <link name="gps">
+  </link>
+  <joint name="gps_base" type="fixed">
+      <origin xyz="0.02 0.0 0.68" rpy="0 0 0"/>
+      <parent link="base_link"/>
+      <child link="gps"/>
+  </joint>
   <!-- IMU sensor description-->
   <xacro:imu_macro prefix="cabot/imu" frame="imu_frame"/>

File: cabot_description/robots/cabot2-gtm.urdf.xacro (robot description, xacro)
@@ -48,4 +48,12 @@
       <child link="lidar_link"/>
     </joint>
+  <!-- add link to gps--> <!-- lidar + 0.1m in z-direction -->
+  <link name="gps">
+  </link>
+  <joint name="gps_base" type="fixed">
+      <origin xyz="0.13 0.0 0.71" rpy="0 0 0"/>
+      <parent link="base_link"/>
+      <child link="gps"/>
+  </joint>
   <link name="rs1_link">
   </link>

File: mf_localization_mapping/urdf/cabot2-e2.urdf (robot description, URDF)
Before this commit: robot cabot2-e2, 6 links, 5 joints
Links:
- added link gps
Joints:
- added joint gps_joint: type fixed, parent velodyne, child gps, origin xyz=0.0 0.0 0.1 rpy=0.0 0.0 0

File: mf_localization_mapping/urdf/cabot2-gt1.urdf (robot description, URDF)
Before this commit: robot cabot2-gt1, 6 links, 5 joints
Links:
- added link gps
Joints:
- added joint gps_joint: type fixed, parent velodyne, child gps, origin xyz=0.0 0.0 0.1 rpy=0.0 0.0 -1.57

File: mf_localization_mapping/urdf/rover.urdf (robot description, URDF)
Before this commit: robot rover, 4 links, 3 joints
Links:
- added link imu_link
Joints:
- added joint imu_link_joint: type fixed, parent imu, child imu_link, origin xyz=0.0 0.0 0.0 rpy=0.0 0.0 0.0

File: mf_localization_mapping/urdf/tripod.urdf (robot description, URDF)
Before this commit: robot tripod, 4 links, 3 joints
Links:
- added link imu_link
Joints:
- added joint imu_link_joint: type fixed, parent imu, child imu_link, origin xyz=0.0 0.0 0.0 rpy=0.0 0.0 0.0
