Commit message: update cabot2-gt1 urdf in the mapping package
Signed-off-by: Masayuki Murata <muratams@jp.ibm.com>

File: mf_localization_mapping/urdf/cabot2-gt1.urdf (robot description, URDF)
Before this commit: robot cabot2-gt1, 5 links, 4 joints
Links:
- added link imu_link
Joints:
- added joint imu_link_joint: type fixed, parent imu, child imu_link, origin xyz=0.0 0.0 0.0 rpy=0.0 0.0 0.0
